File: pcb-business-card/pbc.sch (EAGLE design)
At the start: 25 parts, among them IC1 NET2272REV1A-BCF, J1 CON2, U1 MEGA32U4-MU, U2 RT9193-33GB, U5 TMP117AIYBGR

Commit message: Created gerbers
Connections:
- net PB6(PCINT6/OC1B/OC4B/ADC13) renamed PB6
- net PB7(PCINT7/OC0A/OC1C/!RTS!) renamed PB7
- net PC6(OC3A/!OC4A!) renamed PC6
- net PC7(ICP3/CLK0/OC4A) renamed PC7
Other:
- moved on the sheet: C1, C2, C3, C4, C5, C6, D1, D2, D3, D4, D5, IC1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

Commit message: Added TP and FID
Parts:
- added FD1, FD2, FD3: FIDUCIAL, EET-Symbols:FIDUCIAL
- added TP1, TP2, TP3, TP4, TP5: TP-B0.635, EET-No-Category:TP-B0.635
Changed lines of the file:
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@@
 <part name="U5" library="Sensor" library_urn="urn:adsk.eagle:library:11396555" deviceset="TMP117AIYBGR" device="" package3d_urn="urn:adsk.eagle:package:13238553/2"/>
 <part name="FRAME1" library="zaan-Symbols" library_urn="urn:adsk.eagle:library:16759578" deviceset="A4L-LOC" device=""/>
+<part name="TP1" library="EET-No-Category" deviceset="TP" device="-B0.635"/>
+<part name="TP2" library="EET-No-Category" deviceset="TP" device="-B0.635"/>
+<part name="TP3" library="EET-No-Category" deviceset="TP" device="-B0.635"/>
+<part name="TP4" library="EET-No-Category" deviceset="TP" device="-B0.635"/>
+<part name="TP5" library="EET-No-Category" deviceset="TP" device="-B0.635"/>
+<part name="FD1" library="EET-Symbols" deviceset="FIDUCIAL" device="" package3d_urn="urn:adsk.eagle:package:25891413/2"/>
+<part name="FD2" library="EET-Symbols" deviceset="FIDUCIAL" device="" package3d_urn="urn:adsk.eagle:package:25891413/2"/>
+<part name="FD3" library="EET-Symbols" deviceset="FIDUCIAL" device="" package3d_urn="urn:adsk.eagle:package:25891413/2"/>
 </parts>
 <sheets>
@@
 <attribute name="CHECKED_BY" x="226.06" y="15.24" size="2.54" layer="94"/>
 </instance>
+<instance part="TP1" gate="G$1" x="281.94" y="78.74" smashed="yes">
+<attribute name="NAME" x="280.67" y="80.518" size="1.778" layer="95" align="center-left"/>
+<attribute name="TP_SIGNAL_NAME" x="283.718" y="77.978" size="1.27" layer="97" align="center-left"/>
+</instance>
+<instance part="TP2" gate="G$1" x="292.1" y="81.28" smashed="yes">
+<attribute name="NAME" x="290.83" y="83.058" size="1.778" layer="95" align="center-left"/>
+<attribute name="TP_SIGNAL_NAME" x="293.878" y="80.518" size="1.27" layer="97" align="center-left"/>
+</instance>
+<instance part="TP3" gate="G$1" x="302.26" y="78.74" smashed="yes">
+<attribute name="NAME" x="300.99" y="80.518" size="1.778" layer="95" align="center-left"/>
+<attribute name="TP_SIGNAL_NAME" x="304.038" y="77.978" size="1.27" layer="97" align="center-left"/>
+</instance>
+<instance part="TP4" gate="G$1" x="317.5" y="78.74" smashed="yes">
+<attribute name="NAME" x="316.23" y="80.518" size="1.778" layer="95" align="center-left"/>
+<attribute name="TP_SIGNAL_NAME" x="319.278" y="77.978" size="1.27" layer="97" align="center-left"/>
+</instance>
+<instance part="TP5" gate="G$1" x="330.2" y="76.2" smashed="yes">
+<attribute name="NAME" x="328.93" y="77.978" size="1.778" layer="95" align="center-left"/>
+<attribute name="TP_SIGNAL_NAME" x="331.978" y="75.438" size="1.27" layer="97" align="center-left"/>
+</instance>
+<instance part="FD1" gate="FD" x="274.32" y="60.96" smashed="yes"/>
+<instance part="FD2" gate="FD" x="287.02" y="55.88" smashed="yes"/>
+<instance part="FD3" gate="FD" x="302.26" y="53.34" smashed="yes"/>
 </instances>
 <busses>
